File: KiCad/DroneV2/DroneV2.sch (KiCad schematic (older format))
At the start: 15 parts, among them U1 GY-80, U2 ARDUINO_MICRO_SHIELD, U3 LM7809CT, U4 Battery_Connector

Commit message: Changing pads width and track's layer
Tracks are now on the bottom copper layer.
Pads are wider (oval) with a smaller hole in the middle
Parts:
- BUZ1: footprint Buzzers_Beepers:MagneticBuzzer_StarMicronics_HMB-06_HMB-12 -> drone-custom:MagneticBuzzer_StarMicronics_HMB-06_HMB-12_custom
- C1, C2: footprint Capacitors_ThroughHole:C_Rect_L7_W2_P5 -> drone-custom:C_Rect_L7_W2_P5_custom
- CH1, CH2, CH3, CH4, ESC1, ESC2, ESC3, ESC4: footprint Pin_Headers:Pin_Header_Straight_1x03 -> drone-custom:Pin_Header_Straight_1x03_custom
- U1: footprint GY-80:GY-80-Footprint -> drone-custom:GY-80-Footprint_wider_pad
- U2: footprint arduino_micro_shield:ARDUINO_MICRO_SHIELD -> drone-custom:ARDUINO_MICRO_SHIELD_custom; symbol ARDUINO_MICRO_SHIELD -> ARDUINO_MICRO_SHIELD-RESCUE-DroneV2
- U3: footprint TO_SOT_Packages_THT:TO-220_Neutral123_Vertical -> drone-custom:TO-220_Neutral123_Vertical_custom
- U4: footprint Pin_Headers:Pin_Header_Angled_1x03 -> drone-custom:Pin_Header_Angled_1x03_custom
Changed lines of the file:
@@
 EESchema Schematic File Version 2
+LIBS:DroneV2-rescue
 LIBS:power
 LIBS:device
@@
 LIBS:esc_afro_30a
 LIBS:Turnigy_8CH_Rx
-LIBS:DroneV2_Cache
 LIBS:DroneV2-cache
 EELAYER 25 0
@@
 $EndDescr
 $Comp
-L ARDUINO_MICRO_SHIELD U2
+L ARDUINO_MICRO_SHIELD-RESCUE-DroneV2 U2
 U 1 1 56DF1795
 P 5525 4200
 F 0 "U2" V 6450 4200 60  0000 C CNN
 F 1 "ARDUINO_MICRO_SHIELD" V 4575 4200 60  0000 C CNN
-F 2 "arduino_micro_shield:ARDUINO_MICRO_SHIELD" H 5925 4150 60  0001 C CNN
+F 2 "drone-custom:ARDUINO_MICRO_SHIELD_custom" H 5925 4150 60  0001 C CNN
 F 3 "" H 5925 4150 60  0000 C CNN
 	1    5525 4200
@@
 F 0 "U1" H 3225 3000 60  0000 C CNN
 F 1 "GY-80" H 3225 1775 60  0000 C CNN
-F 2 "GY-80:GY-80-Footprint" H 3025 2900 60  0001 C CNN
+F 2 "drone-custom:GY-80-Footprint_wider_pad" H 3025 2900 60  0001 C CNN
 F 3 "" H 3025 2900 60  0000 C CNN
 	1    3225 2400
@@
 F 0 "ESC1" H 7475 3800 60  0000 C CNN
 F 1 "ESC_Connecor" H 8350 3800 60  0000 C CNN
-F 2 "Pin_Headers:Pin_Header_Straight_1x03" H 7775 3800 60  0001 C CNN
+F 2 "drone-custom:Pin_Header_Straight_1x03_custom" H 7775 3800 60  0001 C CNN
 F 3 "" H 7775 3800 60  0000 C CNN
 	1    7775 3800
@@
 F 0 "ESC2" H 7475 4350 60  0000 C CNN
 F 1 "ESC_Connecor" H 8350 4350 60  0000 C CNN
-F 2 "Pin_Headers:Pin_Header_Straight_1x03" H 7775 4350 60  0001 C CNN
+F 2 "drone-custom:Pin_Header_Straight_1x03_custom" H 7775 4350 60  0001 C CNN
 F 3 "" H 7775 4350 60  0000 C CNN
 	1    7775 4350
@@
 F 0 "ESC3" H 7475 4900 60  0000 C CNN
 F 1 "ESC_Connecor" H 8350 4900 60  0000 C CNN
-F 2 "Pin_Headers:Pin_Header_Straight_1x03" H 7775 4900 60  0001 C CNN
+F 2 "drone-custom:Pin_Header_Straight_1x03_custom" H 7775 4900 60  0001 C CNN
 F 3 "" H 7775 4900 60  0000 C CNN
 	1    7775 4900
@@
 F 0 "ESC4" H 7475 5450 60  0000 C CNN
 F 1 "ESC_Connecor" H 8350 5450 60  0000 C CNN
-F 2 "Pin_Headers:Pin_Header_Straight_1x03" H 7775 5450 60  0001 C CNN
+F 2 "drone-custom:Pin_Header_Straight_1x03_custom" H 7775 5450 60  0001 C CNN
 F 3 "" H 7775 5450 60  0000 C CNN
 	1    7775 5450
@@
 F 0 "U3" H 6975 2475 50  0000 C CNN
 F 1 "LM7809CT" H 7175 2475 50  0000 L CNN
-F 2 "TO_SOT_Packages_THT:TO-220_Neutral123_Vertical" H 7175 2375 50  0001 C CIN
+F 2 "drone-custom:TO-220_Neutral123_Vertical_custom" H 7175 2375 50  0001 C CIN
 F 3 "" H 7175 2275 50  0000 C CNN
 	1    7175 2275
@@
 F 0 "CH1" H 3450 3800 60  0000 C CNN
 F 1 "Rx_Pin" H 2900 3800 60  0000 C CNN
-F 2 "Pin_Headers:Pin_Header_Straight_1x03" H 3200 3800 60  0001 C CNN
+F 2 "drone-custom:Pin_Header_Straight_1x03_custom" H 3200 3800 60  0001 C CNN
 F 3 "" H 3200 3800 60  0000 C CNN
 	1    3200 3800
@@
 F 0 "CH2" H 3450 4350 60  0000 C CNN
 F 1 "Rx_Pin" H 2900 4350 60  0000 C CNN
-F 2 "Pin_Headers:Pin_Header_Straight_1x03" H 3200 4350 60  0001 C CNN
+F 2 "drone-custom:Pin_Header_Straight_1x03_custom" H 3200 4350 60  0001 C CNN
 F 3 "" H 3200 4350 60  0000 C CNN
 	1    3200 4350
@@
 F 0 "CH3" H 3450 4900 60  0000 C CNN
 F 1 "Rx_Pin" H 2900 4900 60  0000 C CNN
-F 2 "Pin_Headers:Pin_Header_Straight_1x03" H 3200 4900 60  0001 C CNN
+F 2 "drone-custom:Pin_Header_Straight_1x03_custom" H 3200 4900 60  0001 C CNN
 F 3 "" H 3200 4900 60  0000 C CNN
 	1    3200 4900
@@
 F 0 "CH4" H 3450 5450 60  0000 C CNN
 F 1 "Rx_Pin" H 2900 5450 60  0000 C CNN
-F 2 "Pin_Headers:Pin_Header_Straight_1x03" H 3200 5450 60  0001 C CNN
+F 2 "drone-custom:Pin_Header_Straight_1x03_custom" H 3200 5450 60  0001 C CNN
 F 3 "" H 3200 5450 60  0000 C CNN
 	1    3200 5450
@@
 F 0 "C1" H 6750 2475 50  0000 L CNN
 F 1 "C" H 6750 2275 50  0000 L CNN
-F 2 "Capacitors_ThroughHole:C_Rect_L7_W2_P5" H 6763 2225 50  0001 C CNN
+F 2 "drone-custom:C_Rect_L7_W2_P5_custom" H 6763 2225 50  0001 C CNN
 F 3 "" H 6725 2375 50  0000 C CNN
 	1    6725 2375
@@
 F 0 "C2" H 7650 2475 50  0000 L CNN
 F 1 "C" H 7650 2275 50  0000 L CNN
-F 2 "Capacitors_ThroughHole:C_Rect_L7_W2_P5" H 7663 2225 50  0001 C CNN
+F 2 "drone-custom:C_Rect_L7_W2_P5_custom" H 7663 2225 50  0001 C CNN
 F 3 "" H 7625 2375 50  0000 C CNN
 	1    7625 2375
@@
 F 0 "U4" H 8375 1975 60  0000 C CNN
 F 1 "Battery_Connector" H 8375 2725 60  0000 C CNN
-F 2 "Pin_Headers:Pin_Header_Angled_1x03" H 8375 2375 60  0001 C CNN
+F 2 "drone-custom:Pin_Header_Angled_1x03_custom" H 8375 2375 60  0001 C CNN
 F 3 "" H 8375 2375 60  0000 C CNN
 	1    8375 2375
@@
 F 0 "BUZ1" H 4275 2975 60  0000 C CNN
 F 1 "Buzzer" H 4275 3225 60  0000 C CNN
-F 2 "Buzzers_Beepers:MagneticBuzzer_StarMicronics_HMB-06_HMB-12" H 4275 3275 60  0001 C CNN
+F 2 "drone-custom:MagneticBuzzer_StarMicronics_HMB-06_HMB-12_custom" H 4275 3275 60  0001 C CNN
 F 3 "" H 4275 3275 60  0000 C CNN
 	1    4275 3275
